File: Reciever/CapstoneReciever/CapstoneReciever.kicad_sch (KiCad schematic)
At the start: 0 parts

Commit message: Started work on reciever
Parts:
- added C1, C7: 470n, symbol Device:C_Small
- added C10, C9: 10u, symbol Device:C_Small
- added C11: 47n, symbol Device:C_Small
- added C2, C3: 43p, symbol Device:C_Small
- added C4, C5, C6: 100u, symbol Device:C_Small
- added C8: 22u, symbol Device:C_Small
- added J1: Conn_01x04, symbol Connector_Generic:Conn_01x04
- added JP1: Bootsel, symbol Jumper:Jumper_2_Open
- added L1: 3u3, symbol Device:L_Small
- added R1, R3: 100k, symbol Device:R_Small_US
- added R2: 43.5k, symbol Device:R_Small_US
- added U1: LM73606RNPR, RNP30_TEX, symbol LM73606:LM73606RNPR
- added U2: ESP32-WROOM-32UE, RF_Module:ESP32-WROOM-32UE, symbol RF_Module:ESP32-WROOM-32UE
Connections:
- new net: C1.1, L1.2, U1.1 (SW), U1.2 (SW), U1.3 (SW), U1.4 (SW), U1.5 (SW)
- new net: C1.2, U1.6 (CBOOT)
- new net: C3.2, U1.7 (VCC)
- new net: JP1.1 (A), U2.25 (IO0)
- new net +3.3V: C2.1, C4.1, C5.1, C6.1, C7.1, J1.1 (Pin_1), L1.1, R1.1, R3.1
- new net FB: C2.2, R1.2, R2.1, U1.11 (FB)
- new net GND: C10.2, C11.2, C3.1, C4.2, C5.2, C6.2, C7.2, C8.2, C9.2, J1.4 (Pin_4), JP1.2 (B), R2.2, U1.12 (NC), U1.13 (NC), U1.14 (NC), U1.15 (NC), U1.17 (SYNC/MODE), U1.19 (AGND), U1.23 (PGND), U1.24 (PGND), U1.25 (PGND), U1.26 (PGND), U1.27 (NC), U1.28 (NC), U1.29 (NC), U1.30 (NC), U1.31 (EPAD), U1.8 (BIAS)
- new net PGOOD: R3.2, U1.16 (PGOOD)
- new net UART_RX: J1.3 (Pin_3), U2.34 (RXD0/IO3)
- new net UART_TX: J1.2 (Pin_2), U2.35 (TXD0/IO1)
- new net Vin: C10.1, C11.1, C8.1, C9.1, U1.18 (EN), U1.20 (PVIN), U1.21 (PVIN), U1.22 (PVIN)
- no-connect marks 0 -> 2

Commit message: Expanded reciever schematic
Other:
- company: (none) -> UMass Lowell
- title: (none) -> Capstone Reciever
Changed lines of the file:
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@@
 	(generator "eeschema")
 	(generator_version "10.0")
-	(paper "A4")
+	(paper "B")
+	(title_block
+		(title "Capstone Reciever")
+		(date "2026-09-17")
+		(rev "1")
+		(company "UMass Lowell")
+	)
 	(junction
 		(at 115.57 62.23)

Commit message: Added TPS552882RPMR buck-boost for 12V switching rail
Parts:
- added C11, C13: 100n, symbol Device:C_Small
- added C15: 10n, symbol Device:C_Small
- added C17: 15p, symbol Device:C_Small
- added C18: 150u, symbol Device:C_Small
- added C2, C5: 68u, symbol Device:C_Polarized_Small_US
- added C20: 10u, symbol Device:C_Polarized_Small_US
- added C21: 4u7, symbol Device:C_Small
- added C8: 10u, symbol Device:C_Small
- added L2: 8u2, symbol Device:L_Small
- added Q1, Q2: CSD18502Q5B, Package_TO_SOT_SMD:TDSON-8-1, symbol Transistor_FET:CSD18502Q5B
- added R10, R9: 1, symbol Device:R_Small_US
- added R11: 35k, symbol Device:R_Small_US
- added R12: 16k, symbol Device:R_Small_US
- added R13, R3, R4, R7: 100k, symbol Device:R_Small_US
- added R14: 11k, symbol Device:R_Small_US
- added R6: 635k, symbol Device:R_Small_US
- added R8: 50k, symbol Device:R_Small_US
- added U2: TPS552882RPMR, RPM0026A-MFG, symbol TPS552882RPMR:TPS552882RPMR
- renumbered C4 to C1, C1 to C10, C8 to C12, C9 to C14, C10 to C16, C11 to C19, C2 to C3, C5 to C4, C3 to C9, R3 to R5, U2 to U3
Connections:
- net GND: now also C17.2, C18.2, C2.2, C20.2, C21.2, C5.2, C8.2, Q2.1 (S), Q2.2 (S), Q2.3 (S), R11.2, R12.2, R14.2, R3.2, R8.2, U2.10 (AGND), U2.15 (MODE), U2.24 (PGND), U2.7 (DITH_SYNC), U2.9 (PGND)
- net Vin renamed +BATT
- net +BATT: now also C2.1, C5.1, C8.1, Q1.5 (D), R6.1, U2.3 (VIN)
- new net: Q2.4 (G), R10.1
- new net: C11.2, L2.1, Q1.1 (S), Q1.2 (S), Q1.3 (S), Q2.5 (D), U2.23 (SW1)
- new net: R13.2, R14.1, U2.14 (FB)
- new net: C11.1, U2.22 (BOOT1)
- new net: R10.2, U2.1 (DR1L)
- new net: R11.1, U2.17 (ILIM)
- new net: C15.1, C17.1, U2.18 (COMP)
- new net: R9.2, U2.2 (DR1H)
- new net: C13.2, U2.20 (BOOT2)
- new net: C13.1, L2.2, U2.21 (SW2), U2.25 (SW2)
- new net: R3.1, R6.2, U2.4 (EN)
- new net: R4.1, U2.5 (PG)
- new net: R7.1, U2.6 (CC_N)
- new net: R8.1, U2.8 (FSW)
- new net: Q1.4 (G), R9.1
- new net: C15.2, R12.1
- new net +12V: C18.1, C20.1, R13.1, U2.11 (VOUT), U2.12 (ISP), U2.13 (ISN), U2.26 (VOUT)
- new net Vcc: C21.1, R4.2, R7.2, U2.19 (VCC)
- no-connect marks 2 -> 3
Other:
- moved on the sheet: J1, JP1, U3
