File: Reciever/CapstoneReciever/CapstoneReciever.kicad_pcb (KiCad board)
At the start: 4 copper layers, 98.2 x 69.1 mm, 39 parts, among them J1 Conn_01x04, J10 C/D, J2 Conn_01x04, J3 Sol1Conn, J4 Sol2Conn, J5 Sol3Conn, J6 Sol4Conn, J7 +12Vin, J8 +3.3Vin, Q1 DMP2035U, Q2 SQD50P04-09L, Q3 CSD18540Q5B, Q4 CSD18540Q5B, Q5 CSD18540Q5B, Q6 CSD18540Q5B, U3 ESP32-WROOM-32UE

Commit message: Added in the solenoid labels, started implementing the endstops. Endstops need pull ups and should be set up for normally closed instead of open for fault protection.
Routing:
- net /DIR/C: track 36.6 -> 41.5 mm
- net /PWM/D: track 36.1 -> 40.0 mm
Other:
- board text added: "Extra"
- board text added: "Main"
- board text added: "Soap"
- board text added: "Sprayers"
Changed lines of the file:
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@@
 	)
 	(footprint "Diode_SMD:D_SMB"
+		(locked yes)
 		(layer "F.Cu")
 		(at 164.070833 107.276666 90)
@@
 	)
 	(footprint "TerminalBlock_CUI:TerminalBlock_CUI_TB007-508-02_1x02_P5.08mm_Horizontal"
+		(locked yes)
 		(layer "F.Cu")
 		(at 153.8 104.459166 -90)
@@
 		)
 	)
+	(gr_text "Sprayers"
+		(at 151 99 0)
+		(layer "F.SilkS")
+		(effects
+			(font
+				(size 1 1)
+				(thickness 0.1)
+			)
+			(justify left bottom)
+		)
+	)
+	(gr_text "Soap\n"
+		(at 151.6 114.6 0)
+		(layer "F.SilkS")
+		(effects
+			(font
+				(size 1 1)
+				(thickness 0.1)
+			)
+			(justify left bottom)
+		)
+	)
+	(gr_text "Main"
+		(at 151.6 129.6 0)
+		(layer "F.SilkS")
+		(effects
+			(font
+				(size 1 1)
+				(thickness 0.1)
+			)
+			(justify left bottom)
+		)
+	)
+	(gr_text "Extra"
+		(at 151.6 132.7 0)
+		(layer "F.SilkS")
+		(effects
+			(font
+				(size 1 1)
+				(thickness 0.1)
+			)
+			(justify left bottom)
+		)
+	)
 	(gr_text "+"
 		(at 190.16 81.2425 0)
@@
 	)
 	(segment
+		(start 188.2 86.8)
+		(end 188.2 97.5)
+		(width 0.5)
+		(layer "F.Cu")
+		(net "Net-(J7-Pin_1)")
+	)
+	(segment
+		(start 188.2 97.5)
+		(end 181.9 97.5)
+		(width 0.5)
+		(layer "F.Cu")
+		(net "Net-(J7-Pin_1)")
+	)
+	(segment
 		(start 178.5675 118.4675)
 		(end 179.75 119.65)
@@
 	)
 	(segment
+		(start 204.7 87.6175)
+		(end 204.7 96.2)
+		(width 0.35)
+		(layer "F.Cu")
+		(net "Net-(J8-Pin_1)")
+	)
+	(segment
+		(start 203.74 86.6575)
+		(end 204.7 87.6175)
+		(width 0.35)
+		(layer "F.Cu")
+		(net "Net-(J8-Pin_1)")
+	)
+	(segment
 		(start 178.015792 124.7675)
 		(end 179.75 126.501708)
@@
 	)
 	(segment
+		(start 202.725 95.15)
+		(end 202.825 95.25)
+		(width 0.35)
+		(layer "F.Cu")
+		(net "Net-(Q1-G)")
+	)
+	(segment
+		(start 198.7 95.15)
+		(end 202.725 95.15)
+		(width 0.35)
+		(layer "F.Cu")
+		(net "Net-(Q1-G)")
+	)
+	(segment
 		(start 164.020278 94.198333)
 		(end 164.132778 94.085833)
@@
 	)
 	(segment
-		(start 228.7 126.5)
-		(end 228.71 126.51)
-		(width 0.127)
+		(start 213.215 118.9)
+		(end 213.205 118.89)
+		(width 0.25)
+		(layer "F.Cu")
+		(net "unconnected-(U3-IO34-Pad6)")
+	)
+	(segment
+		(start 213.245 120.2)
+		(end 213.205 120.16)
+		(width 0.25)
+		(layer "F.Cu")
+		(net "unconnected-(U3-IO35-Pad7)")
+	)
+	(segment
+		(start 208.903375 119.303375)
+		(end 211.03 121.43)
+		(width 0.2)
+		(layer "F.Cu")
+		(net "/Solenoid1Gate")
+	)
+	(segment
+		(start 203.925 119.303375)
+		(end 208.903375 119.303375)
+		(width 0.2)
+		(layer "F.Cu")
+		(net "/Solenoid1Gate")
+	)
+	(segment
+		(start 211.03 121.43)
+		(end 213.205 121.43)
+		(width 0.2)
+		(layer "F.Cu")
+		(net "/Solenoid1Gate")
+	)
+	(segment
+		(start 203.925 124.596708)
+		(end 204.568292 125.24)
+		(width 0.2)
+		(layer "F.Cu")
+		(net "/Solenoid3Gate")
+	)
+	(segment
+		(start 204.568292 125.24)
+		(end 213.205 125.24)
+		(width 0.2)
+		(layer "F.Cu")
+		(net "/Solenoid3Gate")
+	)
+	(segment
+		(start 204.658375 126.51)
+		(end 213.205 126.51)
+		(width 0.2)
+		(layer "F.Cu")
+		(net "/Solenoid4Gate")
+	)
+	(segment
+		(start 203.925 127.243375)
+		(end 204.658375 126.51)
+		(width 0.2)
+		(layer "F.Cu")
+		(net "/Solenoid4Gate")
+	)
+	(segment
+		(start 224.7 126.5)
+		(end 228.7 126.5)
+		(width 0.25)
 		(layer "F.Cu")
 		(net "/DIR{slash}C")
 	)
 	(segment
-		(start 228.71 126.51)
-		(end 230.705 126.51)
-		(width 0.127)
+		(start 228.7 126.5)
+		(end 228.71 126.51)
+		(width 0.25)
 		(layer "F.Cu")
 		(net "/DIR{slash}C")
 	)
 	(segment
-		(start 228.6 126.5)
-		(end 228.7 126.5)
-		(width 0.127)
+		(start 228.71 126.51)
+		(end 230.705 126.51)
+		(width 0.25)
 		(layer "F.Cu")
 		(net "/DIR{slash}C")
 	)
 	(via
-		(at 228.6 126.5)
+		(at 224.7 126.5)
 		(size 0.7)
 		(drill 0.3)
@@
 	)
 	(segment
-		(start 227.7 110.2)
-		(end 227.7 126.2)
-		(width 0.127)
+		(start 226.5 125.6)
+		(end 226.5 111.4)
+		(width 0.25)
 		(layer "B.Cu")
 		(net "/DIR{slash}C")
 	)
 	(segment
-		(start 232.735 94.8575)
-		(end 232.735 105.165)
-		(width 0.127)
+		(start 224.7 126.5)
+		(end 225.6 126.5)
+		(width 0.25)
 		(layer "B.Cu")
 		(net "/DIR{slash}C")
@@
 	(segment
 		(start 232.735 105.165)
-		(end 227.7 110.2)
-		(width 0.127)
+		(end 232.735 94.8575)
+		(width 0.25)
 		(layer "B.Cu")
 		(net "/DIR{slash}C")
 	)
 	(segment
-		(start 227.7 126.2)
-		(end 228 126.5)
-		(width 0.127)
+		(start 225.6 126.5)
+		(end 226.5 125.6)
+		(width 0.25)
 		(layer "B.Cu")
 		(net "/DIR{slash}C")
 	)
 	(segment
-		(start 228 126.5)
-		(end 228.6 126.5)
-		(width 0.127)
+		(start 226.5 111.4)
+		(end 232.735 105.165)
+		(width 0.25)
 		(layer "B.Cu")
 		(net "/DIR{slash}C")
 	)
 	(segment
-		(start 226.84 125.24)
-		(end 230.705 125.24)
+		(start 226.28 125.8)
+		(end 226.84 125.24)
 		(width 0.25)
 		(layer "F.Cu")
@@
 	)
 	(segment
-		(start 226.7 125.1)
-		(end 226.84 125.24)
+		(start 223.6 125.8)
+		(end 226.28 125.8)
+		(width 0.25)
+		(layer "F.Cu")
+		(net "/PWM{slash}D")
+	)
+	(segment
+		(start 226.84 125.24)
+		(end 230.705 125.24)
 		(width 0.25)
 		(layer "F.Cu")
@@
 	)
 	(via
-		(at 226.7 125.1)
+		(at 223.6 125.8)
 		(size 0.7)
 		(drill 0.3)
@@
 	)
 	(segment
-		(start 225.1 123.6)
-		(end 226.6 125.1)
+		(start 223.6 125.8)
+		(end 223.6 125.1)
 		(width 0.25)
 		(layer "B.Cu")
@@
 	)
 	(segment
-		(start 227.655 94.8575)
-		(end 225.1 97.4125)
+		(start 225.9 96.6125)
+		(end 227.655 94.8575)
 		(width 0.25)
 		(layer "B.Cu")
@@
 	)
 	(segment
-		(start 225.1 97.4125)
-		(end 225.1 123.6)
+		(start 225.9 122.8)
+		(end 225.9 96.6125)
 		(width 0.25)
 		(layer "B.Cu")
@@
 	)
 	(segment
-		(start 226.6 125.1)
-		(end 226.7 125.1)
+		(start 223.6 125.1)
+		(end 225.9 122.8)
 		(width 0.25)
 		(layer "B.Cu")
@@
 	)
 	(segment
-		(start 208.903375 119.303375)
-		(end 211.03 121.43)
-		(width 0.2)
-		(layer "F.Cu")
-		(net "/Solenoid1Gate")
-	)
-	(segment
-		(start 203.925 119.303375)
-		(end 208.903375 119.303375)
-		(width 0.2)
-		(layer "F.Cu")
-		(net "/Solenoid1Gate")
-	)
-	(segment
-		(start 211.03 121.43)
-		(end 213.205 121.43)
-		(width 0.2)
-		(layer "F.Cu")
-		(net "/Solenoid1Gate")
-	)
-	(segment
-		(start 203.925 124.596708)
-		(end 204.568292 125.24)
-		(width 0.2)
-		(layer "F.Cu")
-		(net "/Solenoid3Gate")
-	)
-	(segment
-		(start 204.568292 125.24)
-		(end 213.205 125.24)
-		(width 0.2)
-		(layer "F.Cu")
-		(net "/Solenoid3Gate")
-	)
-	(segment
-		(start 204.658375 126.51)
-		(end 213.205 126.51)
-		(width 0.2)
-		(layer "F.Cu")
-		(net "/Solenoid4Gate")
-	)
-	(segment
-		(start 203.925 127.243375)
-		(end 204.658375 126.51)
-		(width 0.2)
-		(layer "F.Cu")
-		(net "/Solenoid4Gate")
-	)
-	(segment
 		(start 188.5 110.945)
 		(end 193.916625 110.945)
@@
 	)
 	(segment
-		(start 188.2 86.8)
-		(end 188.2 97.5)
-		(width 0.5)
-		(layer "F.Cu")
-		(net "Net-(J7-Pin_1)")
-	)
-	(segment
-		(start 188.2 97.5)
-		(end 181.9 97.5)
-		(width 0.5)
-		(layer "F.Cu")
-		(net "Net-(J7-Pin_1)")
-	)
-	(segment
-		(start 204.7 87.6175)
-		(end 204.7 96.2)
-		(width 0.35)
-		(layer "F.Cu")
-		(net "Net-(J8-Pin_1)")
-	)
-	(segment
-		(start 203.74 86.6575)
-		(end 204.7 87.6175)
-		(width 0.35)
-		(layer "F.Cu")
-		(net "Net-(J8-Pin_1)")
-	)
-	(segment
-		(start 202.725 95.15)
-		(end 202.825 95.25)
-		(width 0.35)
-		(layer "F.Cu")
-		(net "Net-(Q1-G)")
-	)
-	(segment
-		(start 198.7 95.15)
-		(end 202.725 95.15)
-		(width 0.35)
-		(layer "F.Cu")
-		(net "Net-(Q1-G)")
-	)
-	(segment
 		(start 178 94.05)
 		(end 180.73 94.05)
@@
 		(net "Net-(Q2-G)")
 	)
-	(segment
-		(start 213.215 118.9)
-		(end 213.205 118.89)
-		(width 0.25)
-		(layer "F.Cu")
-		(net "unconnected-(U3-IO34-Pad6)")
-	)
-	(segment
-		(start 213.245 120.2)
-		(end 213.205 120.16)
-		(width 0.25)
-		(layer "F.Cu")
-		(net "unconnected-(U3-IO35-Pad7)")
-	)
 	(zone
 		(net "GND")
@@
 	)
 	(group ""
+		(locked yes)
 		(members "18709671-84c1-4a82-bd56-cac42606ec9a" "bb11e103-166c-4866-9a2a-e28684cd1921")
 	)

Commit message: Finished routing End of Travel microswitch terminal blocks
Parts:
- added C1: 1000u, Capacitor_SMD:CP_Elec_10x14.3, F.Cu at (159.4, 74.0)
- added C2: 1000u, Capacitor_SMD:CP_Elec_10x14.3, F.Cu at (173.5, 73.8)
- added J11: EoTSwitch2, TerminalBlock_CUI:TerminalBlock_CUI_TB007-508-02_1x02_P5.08mm_Horizontal, F.Cu at (198.2, 138.2)
- added J9: EoTSwitch, TerminalBlock_CUI:TerminalBlock_CUI_TB007-508-02_1x02_P5.08mm_Horizontal, F.Cu at (234.5, 75.7)
- moved J8 19.9 mm to (207.2, 67.1)
- moved J7 19.8 mm to (188.8, 67.1)
- moved REF** 17.5 mm to (221.0, 64.6)
- moved REF** 17.5 mm to (150.0, 64.6)
- moved J10 3.25 mm to (234.2, 97.7), turned to 90 degrees
- moved R6 1.79 mm to (198.9, 96.1), turned to -90 degrees
Connections:
- U3 pad 30: unconnected-(U3-IO18-Pad30) -> /EoT1
- U3 pad 31: unconnected-(U3-IO19-Pad31) -> /EoT2
- U3 pad 33: unconnected-(U3-IO21-Pad33) -> /EoT3
- U3 pad 36: unconnected-(U3-IO22-Pad36) -> /EoT4
Routing:
- net /EoT2: track 0.00 -> 63.6 mm, vias 0 -> 1
- net /EoT1: track 0.00 -> 60.7 mm, vias 0 -> 1
- net /EoT3: track 0.00 -> 44.2 mm, vias 0 -> 1
- net /EoT4: track 0.00 -> 40.5 mm, vias 0 -> 1
- net +12V: track 125.2 -> 149.7 mm
- net Net-(J8-Pin_1): track 9.94 -> 30.2 mm
- net Net-(J7-Pin_1): track 17.0 -> 37.0 mm
- net /PWM/D: track 40.0 -> 48.8 mm
- net /DIR/C: track 41.5 -> 40.0 mm
Other:
- board size 98.2 x 69.1 mm -> 98.2 x 87.1 mm
